File: split_keyboard.kicad_pcb (KiCad board)
At the start: 2 copper layers, 5 x 4.8 mm, 198 parts

Commit message: - Located with exact coordinates the footprints moved.
Parts:
- moved TRRS_R1 7.14 mm to (196.3, 92.2)
- moved SW_R1 6.96 mm to (58.6, 19.2)
- moved SW_L1 5.75 mm to (316.3, 19.2)
- moved BAT_EXT_R1 3.81 mm to (208.2, 48.2)
- moved TRRS_L1 3.76 mm to (178.6, 92.2)
- moved TRRS_R2 2.43 mm to (336.3, 118.2)
- moved BAT_L2 2.16 mm to (38.9, 28.9)
- moved BAT_L1 2.16 mm to (47.0, 28.4)
- moved BAT_R1 2.07 mm to (328.0, 28.4)
- moved BAT_R2 2.07 mm to (336.1, 28.9)
- moved JP_R1 2.02 mm to (218.7, 92.5)
- moved BAT_EXT_L1 1.76 mm to (166.7, 48.2)
- moved TRRS_L2 0.51 mm to (38.6, 118.2)
Other:
- board text added: "EXT -> IC (-11,11)"
- board text added: "Group Ports -> Switch (15,10)"
- board text added: "Switch -> Group Headers (50,0)"
- board text added: "TRRS -> Group of keys (-70,10)"
- board text added: "TRRS -> Group of keys (70,36)"
Changed lines of the file:
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@@
   )
   (footprint "Jumper:SolderJumper-2_P1.3mm_Open_TrianglePad1.0x1.5mm" (layer "F.Cu")
-    (at 220.562 93.218 180)
+    (at 218.694 92.456 180)
     (descr "SMD Solder Jumper, 1x1.5mm Triangular Pads, 0.3mm gap, open")
     (tags "solder jumper open")
@@
     (fp_arc (start -19.901865 15.815496) (mid -19.151865 16.565496) (end -19.901865 17.315496)
       (stroke (width 0.25) (type solid)) (layer "Dwgs.User"))
-    (fp_arc (start -2.503865 17.198296) (mid -3.253839 16.448296) (end -2.503865 15.698295)
+    (fp_arc (start -2.503865 17.198296) (mid -3.253838 16.448296) (end -2.503865 15.698295)
       (stroke (width 0.25) (type solid)) (layer "Dwgs.User"))
     (fp_arc (start -2.503864 17.498295) (mid -3.553865 16.448295) (end -2.503864 15.398295)
@@
   )
   (footprint "Keebio:TRRS-PJ-320A" (layer "F.Cu")
-    (at 338.673 118.872 -90)
+    (at 336.347071 118.161116 -90)
     (property "Arrow Part Number" "PRT-12639")
     (property "Arrow Price/Stock" "https://www.arrow.com/en/products/prt-12639/sparkfun-electronics?region=nac")
@@
     (fp_arc (start -19.901865 15.815496) (mid -19.151865 16.565496) (end -19.901865 17.315496)
       (stroke (width 0.25) (type solid)) (layer "Dwgs.User"))
-    (fp_arc (start -2.503865 17.198296) (mid -3.253839 16.448296) (end -2.503865 15.698295)
+    (fp_arc (start -2.503865 17.198296) (mid -3.253838 16.448296) (end -2.503865 15.698295)
       (stroke (width 0.25) (type solid)) (layer "Dwgs.User"))
     (fp_arc (start -2.503864 17.498295) (mid -3.553865 16.448295) (end -2.503864 15.398295)
@@
   )
   (footprint "JST:JST_PH_B2B-PH-SM4-TB_02x2.00mm_Straight" (layer "F.Cu")
-    (at 166.624 46.482)
+    (at 166.700136 48.244)
     (descr "JST PH series connector, B2B-PH-SM4-TB, top entry type, surface mount, Datasheet: http://www.jst-mfg.com/product/pdf/eng/ePH.pdf")
     (tags "connector jst ph")
@@
   )
   (footprint "Keebio:TRRS-PJ-320A" (layer "F.Cu")
-    (at 203.363 93.472 90)
+    (at 196.347071 92.161116 90)
     (property "Arrow Part Number" "PRT-12639")
     (property "Arrow Price/Stock" "https://www.arrow.com/en/products/prt-12639/sparkfun-electronics?region=nac")
@@
   )
   (footprint "Keebio:TRRS-PJ-320A" (layer "F.Cu")
-    (at 175.1655 93.726 -90)
+    (at 178.585971 92.159637 -90)
     (property "Arrow Part Number" "PRT-12639")
     (property "Arrow Price/Stock" "https://www.arrow.com/en/products/prt-12639/sparkfun-electronics?region=nac")
@@
   )
   (footprint "Keebio:TRRS-PJ-320A" (layer "F.Cu")
-    (at 38.885 117.743 90)
+    (at 38.585971 118.159637 90)
     (property "Arrow Part Number" "PRT-12639")
     (property "Arrow Price/Stock" "https://www.arrow.com/en/products/prt-12639/sparkfun-electronics?region=nac")
@@
   )
   (footprint "JST:JST_PH_B2B-PH-SM4-TB_02x2.00mm_Straight" (layer "F.Cu")
-    (at 208.182 44.432)
+    (at 208.208935 48.241116)
     (descr "JST PH series connector, B2B-PH-SM4-TB, top entry type, surface mount, Datasheet: http://www.jst-mfg.com/product/pdf/eng/ePH.pdf")
     (tags "connector jst ph")
@@
   )
   (footprint "JST:JST_GH_BM02B-GHS-TBT_02x1.25mm_Straight" (layer "B.Cu")
-    (at 335.788 30.967)
+    (at 336.078071 28.916991)
     (descr "JST GH series connector, BM02B-GHS-TBT, top entry type")
     (tags "connector jst GH SMT top vertical entry 1.25mm pitch")
@@
   )
   (footprint "Slide Switch:PCM13SMTR" (layer "B.Cu")
-    (at 310.769 20.574)
+    (at 316.347071 19.161116)
     (descr "PCM13SMTR-3")
     (tags "Switch")
@@
   )
   (footprint "JST:JST_PH_B2B-PH-SM4-TB_02x2.00mm_Straight" (layer "B.Cu")
-    (at 47.498 30.48)
+    (at 46.968471 28.385512)
     (descr "JST PH series connector, B2B-PH-SM4-TB, top entry type, surface mount, Datasheet: http://www.jst-mfg.com/product/pdf/eng/ePH.pdf")
     (tags "connector jst ph")
@@
   )
   (footprint "Slide Switch:PCM13SMTR" (layer "B.Cu")
-    (at 65.335 20.879)
+    (at 58.585971 19.159637)
     (descr "PCM13SMTR-3")
     (tags "Switch")
@@
   )
   (footprint "JST:JST_GH_BM02B-GHS-TBT_02x1.25mm_Straight" (layer "B.Cu")
-    (at 39.383 31.01)
+    (at 38.853471 28.915512)
     (descr "JST GH series connector, BM02B-GHS-TBT, top entry type")
     (tags "connector jst GH SMT top vertical entry 1.25mm pitch")
@@
   )
   (footprint "JST:JST_PH_B2B-PH-SM4-TB_02x2.00mm_Straight" (layer "B.Cu")
-    (at 327.676 30.437)
+    (at 327.966071 28.386991)
     (descr "JST PH series connector, B2B-PH-SM4-TB, top entry type, surface mount, Datasheet: http://www.jst-mfg.com/product/pdf/eng/ePH.pdf")
     (tags "connector jst ph")
@@
     (effects (font (size 1 1) (thickness 0.15)) (justify left bottom))
   )
+  (gr_text "EXT -> IC\n(-11,11)" (at 204.978 56.007) (layer "Cmts.User")
+    (effects (font (size 1 1) (thickness 0.15)) (justify left bottom))
+  )
+  (gr_text "TRRS -> Group of keys\n(70,36)" (at 321.056 125.095) (layer "Cmts.User")
+    (effects (font (size 1 1) (thickness 0.15)) (justify left bottom))
+  )
   (gr_text "IC -> Pin24\n(0,-10)" (at 215.138 43.18) (layer "Cmts.User")
     (effects (font (size 1 1) (thickness 0.15)) (justify left bottom))
@@
     (effects (font (size 1 1) (thickness 0.15)) (justify left bottom))
   )
+  (gr_text "Switch -> Group Headers \n(50,0)" (at 307.34 14.859) (layer "Cmts.User")
+    (effects (font (size 1 1) (thickness 0.15) italic) (justify left bottom))
+  )
   (gr_text "MCU -> Group of keys\n(-70,-40)" (at 194.945 87.503) (layer "Cmts.User")
     (effects (font (size 1 1) (thickness 0.15)) (justify left bottom))
   )
-  (gr_text "Group Headers -> Group of keys\n(0,-63)" (at 294.132 19.939) (layer "Cmts.User")
+  (gr_text "TRRS -> Group of keys\n(-70,10)" (at 195.834 99.187) (layer "Cmts.User")
+    (effects (font (size 1 1) (thickness 0.15)) (justify left bottom))
+  )
+  (gr_text "Group Ports -> Switch\n(15,10)" (at 341.503 29.337) (layer "Cmts.User")
+    (effects (font (size 1 1) (thickness 0.15)) (justify left bottom))
+  )
+  (gr_text "Group Headers -> Group of keys\n(0,-63)" (at 266.7 15.875) (layer "Cmts.User")
     (effects (font (size 1 1) (thickness 0.15)) (justify left bottom))
   )

Commit message: added more components and fix some in sch
Parts:
- removed C5, C6, C7, C8: 10uf, Capacitor_SMD:C_0805_2012Metric
- removed TRRS_R1, TRRS_R2: PRT-12639, Keebio:TRRS-PJ-320A
- added L_R1: 10k, Resistor_SMD:R_0805_2012Metric, F.Cu at (206.0, 171.2)
- added L_R2: 10k, Resistor_SMD:R_0805_2012Metric, F.Cu at (206.0, 174.2)
- added R_C1: 10uf, Capacitor_SMD:C_0805_2012Metric, F.Cu at (201.5, 157.9)
- added R_C2: 10uf, Capacitor_SMD:C_0805_2012Metric, F.Cu at (201.5, 160.9)
- added R_C3: 10uf, Capacitor_SMD:C_0805_2012Metric, F.Cu at (201.5, 164.0)
- added R_C4: 10uf, Capacitor_SMD:C_0805_2012Metric, F.Cu at (201.5, 167.0)
- added R_C5: 10uf, Capacitor_SMD:C_0805_2012Metric, F.Cu at (201.5, 170.0)
- added R_C6: 10uf, Capacitor_SMD:C_0805_2012Metric, F.Cu at (201.5, 173.0)
- added R_J1: Qwiic_RA, SparkFun-Connector:JST_SMD_1.0mm-4_RA, F.Cu at (207.8, 157.8)
- added R_J2: Qwiic_RA, SparkFun-Connector:JST_SMD_1.0mm-4_RA, F.Cu at (207.8, 164.4)
- added R_R1: 10k, Resistor_SMD:R_0805_2012Metric, F.Cu at (206.0, 177.1)
- added R_R2: 10k, Resistor_SMD:R_0805_2012Metric, F.Cu at (206.0, 180.1)
- added R_TRRS1: PRT-12639, Keebio:TRRS-PJ-320A, F.Cu at (196.3, 92.2)
- added R_TRRS2: PRT-12639, Keebio:TRRS-PJ-320A, F.Cu at (336.3, 118.2)
Connections:
- net +3.3V_LEFT renamed +3.3V
- net +3.3V_RIGHT renamed +3.3VA
- net +5V_LEFT renamed +5V
- net +5V_RIGHT renamed +5VA
- net IO_INT_L renamed L_IO_INT
- net IO_INT_R renamed R_IO_INT
- net VBAT_R renamed R_VBAT
- net VLED_R renamed R_VLED
- IO_L1 pad 20: unconnected-(IO_L1-~{RESET}-Pad20) -> Net-(IO_L1-~{RESET})
- IO_R1 pad 20: unconnected-(IO_R1-~{RESET}-Pad20) -> Net-(IO_R1-~{RESET})
- T-Display-S3_R1 pad 3: LED_OUT_R -> R_LED_OUT
Routing:
- net Net-(R_D16-A): track 0.00 -> 7.51 mm
- net Net-(R_D14-A): track 0.00 -> 7.51 mm
- net Net-(R_D11-A): track 0.00 -> 7.51 mm
- net Net-(R_D10-A): track 0.00 -> 7.42 mm
- net Net-(R_D9-A): track 0.00 -> 7.42 mm
- net Net-(R_D15-A): track 0.00 -> 7.42 mm

Commit message: Right side almost done
Parts:
- removed R_C6: 10uf, Capacitor_SMD:C_0805_2012Metric
- removed R_J2: Qwiic_RA, SparkFun-Connector:JST_SMD_1.0mm-4_RA
- removed R_TRRS2, TRRS_L2: PRT-12639, Keebio:TRRS-PJ-320A
- added L_C5: 10uf, Capacitor_SMD:C_0805_2012Metric, B.Cu at (165.4, 33.3)
- added L_J1: Qwiic_RA, SparkFun-Connector:JST_SMD_1.0mm-4_RA, F.Cu at (175.6, 102.2)
- L_R1, L_R2, R_C1, R_C2, R_C3, R_C4, R_C5, R_R1, R_R2: moved to B.Cu
- moved R_C1 177.0 mm to (336.0, 42.9)
- moved R_C3 158.1 mm to (336.0, 80.9)
- moved R_R2 142.0 mm to (211.5, 38.2), turned to -90 degrees
- moved R_R1 141.9 mm to (214.9, 35.6)
- moved L_R1 140.3 mm to (165.4, 37.0), turned to 180 degrees
- moved L_R2 140.3 mm to (165.4, 39.9), turned to 180 degrees
- moved R_C5 132.3 mm to (213.9, 38.2), turned to -90 degrees
- moved R_C2 113.6 mm to (229.8, 50.9), turned to 180 degrees
- moved R_C4 82.9 mm to (229.9, 89.0), turned to 180 degrees
- moved R_J1 56.3 mm to (199.3, 102.2), turned to -90 degrees
- moved H_R1 28.1 mm to (104.5, 171.7)
- moved JP_R1 2.37 mm to (216.3, 92.2)
Routing:
- net R_KEY_COL1: track 64.3 -> 229.3 mm, vias 0 -> 1
- net R_KEY_ROW1: track 104.5 -> 231.2 mm, vias 0 -> 2
- net R_KEY_COL2: track 64.2 -> 169.8 mm, vias 0 -> 1
- net R_KEY_COL8: track 0.00 -> 102.9 mm, vias 0 -> 1
- net R_KEY_COL7: track 0.00 -> 86.7 mm, vias 0 -> 1
- net R_KEY_COL3: track 64.2 -> 146.8 mm, vias 0 -> 1
- net R_KEY_COL4: track 64.2 -> 121.6 mm, vias 0 -> 1
- net R_SCL: track 0.00 -> 55.2 mm
- net R_SDA: track 0.00 -> 51.5 mm
- net R_KEY_ROW2: track 104.5 -> 150.2 mm
- net GND: track 598.1 -> 636.6 mm
- net R_KEY_COL5: track 64.2 -> 100.5 mm, vias 0 -> 1
- net +3.3VA: track 0.00 -> 35.6 mm
- net R_KEY_ROW3: track 104.5 -> 132.1 mm, vias 0 -> 2
- net Net-(JP_R1-B): track 0.00 -> 22.7 mm
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Other:
- board text added: "Jumper -> Group of keys (-50,10)"
- board text added: "QWIIC -> Group of keys (-67,20)"
- board text removed: "TRRS -> Group of keys (70,36)"

Commit message: -Almost done
Parts:
- R_TRRS1, TRRS_L1: footprint Keebio:TRRS-PJ-320A -> custom:TRRS-PJ-320A
- moved SW_R1 257.9 mm to (316.5, 18.5)
- moved SW_L1 257.8 mm to (58.6, 19.2)
- moved L_C5 8.08 mm to (168.4, 40.8)
- moved L_R1 5.56 mm to (170.9, 37.2), turned to -90 degrees
- moved L_R2 3.93 mm to (167.0, 36.3)
- turned IO_L1 to 90 degrees
- turned JP_R2 to 180 degrees
Connections:
- L_SW1 pad 1: L_KEY_COL2 -> L_KEY_COL3
- L_SW10 pad 1: L_KEY_COL4 -> L_KEY_COL5
- L_SW11 pad 1: L_KEY_COL3 -> L_KEY_COL4
- L_SW12 pad 1: L_KEY_COL2 -> L_KEY_COL3
- L_SW13 pad 1: L_KEY_COL2 -> L_KEY_COL3
- L_SW14 pad 1: L_KEY_COL3 -> L_KEY_COL4
- L_SW15 pad 1: L_KEY_COL4 -> L_KEY_COL5
- L_SW16 pad 1: L_KEY_COL5 -> L_KEY_COL6
- L_SW17 pad 1: L_KEY_COL6 -> L_KEY_COL7
- L_SW18 pad 1: L_KEY_COL7 -> L_KEY_COL8
- L_SW19 pad 1: L_KEY_COL7 -> L_KEY_COL8
- L_SW2 pad 1: L_KEY_COL3 -> L_KEY_COL4
- L_SW20 pad 1: L_KEY_COL6 -> L_KEY_COL7
- L_SW21 pad 1: L_KEY_COL5 -> L_KEY_COL6
- L_SW22 pad 1: L_KEY_COL4 -> L_KEY_COL5
- L_SW23 pad 1: L_KEY_COL3 -> L_KEY_COL4
- L_SW24 pad 1: L_KEY_COL2 -> L_KEY_COL3
- L_SW25 pad 1: L_KEY_COL1 -> L_KEY_COL2
- L_SW26 pad 1: L_KEY_COL8 -> L_KEY_COL1
- L_SW3 pad 1: L_KEY_COL4 -> L_KEY_COL5
- L_SW4 pad 1: L_KEY_COL5 -> L_KEY_COL6
- L_SW5 pad 1: L_KEY_COL6 -> L_KEY_COL7
- L_SW6 pad 1: L_KEY_COL7 -> L_KEY_COL8
- L_SW7 pad 1: L_KEY_COL7 -> L_KEY_COL8
- L_SW8 pad 1: L_KEY_COL6 -> L_KEY_COL7
- L_SW9 pad 1: L_KEY_COL5 -> L_KEY_COL6
- T-Display-S3_L1 pad 1: unconnected-(T-Display-S3_L1-3v-Pad1) -> +3.3V
Routing:
- net L_KEY_COL8: track 0.00 -> 187.7 mm, vias 0 -> 1
- net Net-(BAT_EXT_R1-Pin_2): track 0.00 -> 167.8 mm, vias 0 -> 1
- net R_VBAT: track 0.00 -> 142.5 mm, vias 0 -> 1
- net R_U1_TXD: track 0.00 -> 123.7 mm
- net R_U1_RXD: track 0.00 -> 123.0 mm
- net R_SPI_CS: track 0.00 -> 105.6 mm
- net L_KEY_COL1: track 0.00 -> 105.1 mm, vias 0 -> 1
- net R_SPI_D: track 0.00 -> 100.7 mm
- net L_KEY_COL7: track 64.2 -> 164.9 mm, vias 0 -> 1
- net R_SPI_CLK: track 0.00 -> 95.9 mm
- net R_KEY_COL9: track 0.00 -> 91.7 mm, vias 0 -> 2
- net R_SPI_Q: track 0.00 -> 91.1 mm
- net L_SDA: track 0.00 -> 88.7 mm
- net R_KEY_COL10: track 0.00 -> 87.7 mm, vias 0 -> 2
- net L_SCL: track 0.00 -> 87.7 mm
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
Commit message: added outline and holes
Parts:
- moved H_R2 280.8 mm to (336.6, 20.8)
- moved H_R1 239.8 mm to (337.3, 114.1)
- moved H_R3 175.3 mm to (195.6, 21.3)
- moved H_L3 169.5 mm to (178.4, 21.0)
- moved H_R4 151.1 mm to (207.5, 73.2)
- moved H_L2 141.2 mm to (38.1, 20.6)
- moved H_L4 126.9 mm to (166.9, 72.3)
- moved H_R5 123.5 mm to (196.8, 112.8)
- moved H_L5 112.0 mm to (176.7, 112.5)
- moved H_L1 57.2 mm to (37.6, 113.2)
- moved L_R1 10.9 mm to (160.1, 38.9), turned to 180 degrees
- moved L_C5 8.52 mm to (161.3, 36.1), turned to 90 degrees
- moved L_R2 3.31 mm to (163.7, 36.1), turned to 90 degrees
- moved R_SWB1 0.66 mm to (316.5, 19.2)
- moved L_JP2 0.29 mm to (132.0, 18.2), turned to 0 degrees
- renumbered BAT_L1 to L_BAT1, BAT_L2 to L_BAT2, BAT_EXT_L1 to L_BAT_EXT1, C1 to L_C1, C2 to L_C2, C3 to L_C3, C4 to L_C4, IO_L1 to L_IO1, IOExp_Pinout_L1 to L_IOExp_Pinout1, JP_L1 to L_JP1, JP_L2 to L_JP2, S3_Pinout_L1 to L_S3_Pinout1, SW_L1 to L_SWB1, T-Display-S3_L1 to L_T-Display-S3, BAT_R1 to R_BAT1, BAT_R2 to R_BAT2, BAT_EXT_R1 to R_BAT_EXT1, IO_R1 to R_IO1, IOExp_Pinout_R1 to R_IOExp_Pinout1, JP_R1 to R_JP1, JP_R2 to R_JP2, S3_Pinout_R1 to R_S3_Pinout1, SW_R1 to R_SWB1, T-Display-S3_R1 to R_T-Display-S3
Connections:
- net +3.3V renamed L_+3.3V
- net +3.3VA renamed R_+3.3V
- net +5V renamed L_+5V
- net +5VA renamed R_+5V
- net GND renamed R_GND
- net GND1 renamed R_GND1
- net GND2 renamed L_GND
- net GND3 renamed L_GND1
- net LED_OUT_L renamed L_LED_OUT
- net VBAT_L renamed L_VBAT
- net VLED_L renamed L_VLED
- R_LED1 pad 4: LED_OUT_R -> R_LED_OUT
Routing:
- net Net-(L_BAT1-Pin_2): track 0.00 -> 162.3 mm, vias 0 -> 1
- net L_VBAT: track 0.00 -> 138.1 mm, vias 0 -> 3
- net L_GND: track 656.4 -> 781.7 mm, vias 4 -> 10
- net L_U1_TXD: track 0.00 -> 107.7 mm, vias 0 -> 1
- net L_U1_RXD: track 0.00 -> 107.4 mm, vias 0 -> 1
- net L_KEY_ROW5: track 0.00 -> 96.3 mm, vias 0 -> 2
- net L_KEY_ROW6: track 0.00 -> 91.0 mm, vias 0 -> 2
- net L_KEY_COL9: track 0.95 -> 90.3 mm, vias 1 -> 4
- net L_SPI_CS: track 0.00 -> 87.1 mm, vias 0 -> 1
- net L_KEY_COL10: track 0.00 -> 86.1 mm, vias 0 -> 4
- net L_KEY_ROW7: track 0.00 -> 85.9 mm, vias 0 -> 2
- net R_LED_OUT: track 0.00 -> 85.1 mm, vias 0 -> 1
- net L_SPI_D: track 0.00 -> 81.7 mm, vias 0 -> 1
- net L_KEY_ROW8: track 0.00 -> 80.5 mm, vias 0 -> 2
- net L_SPI_CLK: track 0.00 -> 76.0 mm, vias 0 -> 1
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Other:
- board size 5 x 4.8 mm -> 307.5 x 126.2 mm
- board text added: "H1 -> Group of keys (71,35)"
