File: split_keyboard.kicad_sch (KiCad schematic)
At the start: 198 parts

Commit message: - Made a custom form of the key - Brang back the MINI-E lib, it was used for sch
Signed-off-by: Pablo Oyarzo <pabloantoyarzo@gmail.com>
Parts:
- L_SW1, L_SW10, L_SW11, L_SW12, L_SW13, L_SW14, L_SW15, L_SW16, L_SW17, L_SW18, L_SW19, L_SW2, L_SW20, L_SW21, L_SW22, L_SW23, L_SW24, L_SW25, L_SW26, L_SW3, L_SW4, L_SW5, L_SW6, L_SW7, L_SW8, L_SW9, R_SW1, R_SW10, R_SW11, R_SW12, R_SW13, R_SW14, R_SW15, R_SW16, R_SW17, R_SW18, R_SW19, R_SW2, R_SW20, R_SW21, R_SW22, R_SW23, R_SW24, R_SW25, R_SW26, R_SW3, R_SW4, R_SW5, R_SW6, R_SW7, R_SW8, R_SW9: footprint Keyswitches:Kailh_socket_MX -> custom:SW_Hotswap_Kailh_Choc_V1V2_Plated_1.00u
- TRRS_L1, TRRS_L2, TRRS_R1, TRRS_R2: footprint TRRS:PRT12639 -> Keebio:TRRS-PJ-320A
Connections:
- net VBAT_L: now also SW_L1.3 (COM); no longer SW_L1.1 (NO_1)
- net VBAT_R: now also SW_R1.3 (COM); no longer SW_R1.1 (NO_1)
- net at BAT_R1.1 (Pin_1), BAT_R2.1 (Pin_1): now also SW_R1.4 (NO_2); no longer SW_R1.3 (COM)
- net at BAT_L1.1 (Pin_1), BAT_L2.1 (Pin_1): now also SW_L1.4 (NO_2); no longer SW_L1.3 (COM)
- no-connect marks 31 -> 29

Commit message: - Changed files for next version's keyboard layout - Added instructions on how to use kb's layout file - Modified a bit the LED footprint - Modified all names for symbols and part inside the pcb and sch for switches, leds and diodes
Parts:
- removed D27, D28, D29, D30, D31, D32, D33, D34, D35, D36, D37, D38, D39, D40, D41, D42, D43, D44, D45, D46, D47, D48, D49, D50, D51, D52: D, custom:D_0805, symbol Device:D
- removed LED_L10, LED_L11, LED_L12, LED_L13, LED_L14, LED_L15, LED_L16, LED_L17, LED_L18, LED_L19, LED_L2, LED_L20, LED_L21, LED_L22, LED_L23, LED_L24, LED_L25, LED_L26, LED_L3, LED_L4, LED_L5, LED_L6, LED_L7, LED_L8, LED_L9, LED_R10, LED_R11, LED_R12, LED_R13, LED_R14, LED_R15, LED_R16, LED_R17, LED_R18, LED_R19, LED_R2, LED_R20, LED_R21, LED_R22, LED_R23, LED_R24, LED_R25, LED_R26, LED_R3, LED_R4, LED_R5, LED_R6, LED_R7, LED_R8, LED_R9: SK6812MINI-E, custom:SK6812-MINI-E, symbol LED:SK6812MINI-E
- added L_LED10, L_LED11, L_LED12, L_LED13, L_LED14, L_LED15, L_LED16, L_LED17, L_LED18, L_LED19, L_LED2, L_LED20, L_LED21, L_LED22, L_LED23, L_LED24, L_LED25, L_LED26, L_LED3, L_LED4, L_LED5, L_LED6, L_LED7, L_LED8, L_LED9, R_LED10, R_LED11, R_LED12, R_LED13, R_LED14, R_LED15, R_LED16, R_LED17, R_LED18, R_LED19, R_LED2, R_LED20, R_LED21, R_LED22, R_LED23, R_LED24, R_LED25, R_LED26, R_LED3, R_LED4, R_LED5, R_LED6, R_LED7, R_LED8, R_LED9: SK6812MINI-E, custom:SK6812-MINI-E, symbol LED:SK6812MINI-E
- added R_D1, R_D10, R_D11, R_D12, R_D13, R_D14, R_D15, R_D16, R_D17, R_D18, R_D19, R_D2, R_D20, R_D21, R_D22, R_D23, R_D24, R_D25, R_D26, R_D3, R_D4, R_D5, R_D6, R_D7, R_D8, R_D9: D, custom:D_0805, symbol Device:D
- renumbered D1 to L_D1, D14 to L_D10, D18 to L_D11, D22 to L_D12, D3 to L_D13, D7 to L_D14, D11 to L_D15, D15 to L_D16, D19 to L_D17, D23 to L_D18, D4 to L_D19, D5 to L_D2, D8 to L_D20, D12 to L_D21, D16 to L_D22, D20 to L_D23, D24 to L_D24, D25 to L_D25, D26 to L_D26, D9 to L_D3, D13 to L_D4, D17 to L_D5, D21 to L_D6, D2 to L_D7, D6 to L_D8, D10 to L_D9, LED_L1 to L_LED1, L_SW14 to L_SW10, L_SW18 to L_SW11, L_SW22 to L_SW12, L_SW3 to L_SW13, L_SW7 to L_SW14, L_SW11 to L_SW15, L_SW15 to L_SW16, L_SW19 to L_SW17, L_SW23 to L_SW18, L_SW4 to L_SW19, L_SW5 to L_SW2, L_SW8 to L_SW20, L_SW12 to L_SW21, L_SW16 to L_SW22, L_SW20 to L_SW23, L_SW9 to L_SW3, L_SW13 to L_SW4, L_SW17 to L_SW5, L_SW21 to L_SW6, L_SW2 to L_SW7, L_SW6 to L_SW8, L_SW10 to L_SW9, LED_R1 to R_LED1
Connections:
- net GND: now also R_LED10.3 (GND), R_LED11.3 (GND), R_LED12.3 (GND), R_LED13.3 (GND), R_LED14.3 (GND), R_LED15.3 (GND), R_LED16.3 (GND), R_LED17.3 (GND), R_LED18.3 (GND), R_LED19.3 (GND), R_LED2.3 (GND), R_LED20.3 (GND), R_LED21.3 (GND), R_LED22.3 (GND), R_LED23.3 (GND), R_LED24.3 (GND), R_LED25.3 (GND), R_LED26.3 (GND), R_LED3.3 (GND), R_LED4.3 (GND), R_LED5.3 (GND), R_LED6.3 (GND), R_LED7.3 (GND), R_LED8.3 (GND), R_LED9.3 (GND)
- net GND2: now also L_LED10.3 (GND), L_LED11.3 (GND), L_LED12.3 (GND), L_LED13.3 (GND), L_LED14.3 (GND), L_LED15.3 (GND), L_LED16.3 (GND), L_LED17.3 (GND), L_LED18.3 (GND), L_LED19.3 (GND), L_LED2.3 (GND), L_LED20.3 (GND), L_LED21.3 (GND), L_LED22.3 (GND), L_LED23.3 (GND), L_LED24.3 (GND), L_LED25.3 (GND), L_LED26.3 (GND), L_LED3.3 (GND), L_LED4.3 (GND), L_LED5.3 (GND), L_LED6.3 (GND), L_LED7.3 (GND), L_LED8.3 (GND), L_LED9.3 (GND)
- net L_KEY_COL1: now also L_SW25.1; no longer L_D26.1 (K)
- net L_KEY_COL2: now also L_SW12.1, L_SW18.1, L_SW24.1, L_SW6.1; no longer L_D25.1 (K)
- net L_KEY_COL3: now also L_SW11.1, L_SW17.1, L_SW23.1, L_SW5.1; no longer L_D12.1 (K), L_D18.1 (K), L_D24.1 (K), L_D6.1 (K)
- net L_KEY_COL4: now also L_SW10.1, L_SW16.1, L_SW22.1, L_SW4.1; no longer L_D11.1 (K), L_D17.1 (K), L_D23.1 (K), L_D5.1 (K)
- net L_KEY_COL5: now also L_SW15.1, L_SW21.1, L_SW3.1, L_SW9.1; no longer L_D10.1 (K), L_D16.1 (K), L_D22.1 (K), L_D4.1 (K)
- net L_KEY_COL6: now also L_SW14.1, L_SW2.1, L_SW20.1, L_SW8.1; no longer L_D15.1 (K), L_D21.1 (K), L_D3.1 (K), L_D9.1 (K)
- net L_KEY_COL7: now also L_SW1.1, L_SW13.1, L_SW19.1, L_SW7.1; no longer L_D14.1 (K), L_D2.1 (K), L_D20.1 (K), L_D8.1 (K)
- net L_KEY_COL8: now also L_SW26.1; no longer L_D1.1 (K), L_D13.1 (K), L_D19.1 (K), L_D7.1 (K)
- net L_KEY_ROW1: now also L_D1.1 (K), L_D2.1 (K), L_D3.1 (K), L_D4.1 (K), L_D5.1 (K), L_D6.1 (K); no longer L_SW1.2, L_SW2.2, L_SW3.2, L_SW4.2, L_SW5.2, L_SW6.2
- net L_KEY_ROW2: now also L_D10.1 (K), L_D11.1 (K), L_D12.1 (K), L_D7.1 (K), L_D8.1 (K), L_D9.1 (K); no longer L_SW10.2, L_SW11.2, L_SW12.2, L_SW7.2, L_SW8.2, L_SW9.2
- net L_KEY_ROW3: now also L_D13.1 (K), L_D14.1 (K), L_D15.1 (K), L_D16.1 (K), L_D17.1 (K), L_D18.1 (K); no longer L_SW13.2, L_SW14.2, L_SW15.2, L_SW16.2, L_SW17.2, L_SW18.2
- net L_KEY_ROW4: now also L_D19.1 (K), L_D20.1 (K), L_D21.1 (K), L_D22.1 (K), L_D23.1 (K), L_D24.1 (K), L_D25.1 (K), L_D26.1 (K); no longer L_SW19.2, L_SW20.2, L_SW21.2, L_SW22.2, L_SW23.2, L_SW24.2, L_SW25.2, L_SW26.2
- net R_KEY_COL1: now also R_SW12.1, R_SW18.1, R_SW26.1, R_SW6.1
- net R_KEY_COL2: now also R_SW11.1, R_SW17.1, R_SW25.1, R_SW5.1
- net R_KEY_COL3: now also R_SW10.1, R_SW16.1, R_SW24.1, R_SW4.1
- net R_KEY_COL4: now also R_SW15.1, R_SW23.1, R_SW3.1, R_SW9.1
- net R_KEY_COL5: now also R_SW14.1, R_SW2.1, R_SW22.1, R_SW8.1
- net R_KEY_COL6: now also R_SW1.1, R_SW13.1, R_SW21.1, R_SW7.1
- net R_KEY_COL7: now also R_SW20.1
- net R_KEY_COL8: now also R_SW19.1
- net R_KEY_ROW1: now also R_D19.1 (K), R_D20.1 (K), R_D21.1 (K), R_D22.1 (K), R_D23.1 (K), R_D24.1 (K), R_D25.1 (K), R_D26.1 (K); no longer R_SW1.2, R_SW10.2, R_SW14.2, R_SW18.2, R_SW2.2, R_SW22.2, R_SW26.2, R_SW6.2
- net R_KEY_ROW2: now also R_D13.1 (K), R_D14.1 (K), R_D15.1 (K), R_D16.1 (K), R_D17.1 (K), R_D18.1 (K); no longer R_SW13.2, R_SW17.2, R_SW21.2, R_SW25.2, R_SW5.2, R_SW9.2
- net R_KEY_ROW3: now also R_D10.1 (K), R_D11.1 (K), R_D12.1 (K), R_D7.1 (K), R_D8.1 (K), R_D9.1 (K); no longer R_SW12.2, R_SW16.2, R_SW20.2, R_SW24.2, R_SW4.2, R_SW8.2
- net R_KEY_ROW4: now also R_D1.1 (K), R_D2.1 (K), R_D3.1 (K), R_D4.1 (K), R_D5.1 (K), R_D6.1 (K); no longer R_SW11.2, R_SW15.2, R_SW19.2, R_SW23.2, R_SW3.2, R_SW7.2
- net VLED_L: now also L_LED10.1 (VDD), L_LED11.1 (VDD), L_LED12.1 (VDD), L_LED13.1 (VDD), L_LED14.1 (VDD), L_LED15.1 (VDD), L_LED16.1 (VDD), L_LED17.1 (VDD), L_LED18.1 (VDD), L_LED19.1 (VDD), L_LED2.1 (VDD), L_LED20.1 (VDD), L_LED21.1 (VDD), L_LED22.1 (VDD), L_LED23.1 (VDD), L_LED24.1 (VDD), L_LED25.1 (VDD), L_LED26.1 (VDD), L_LED3.1 (VDD), L_LED4.1 (VDD), L_LED5.1 (VDD), L_LED6.1 (VDD), L_LED7.1 (VDD), L_LED8.1 (VDD), L_LED9.1 (VDD)
- net VLED_R: now also R_LED10.1 (VDD), R_LED11.1 (VDD), R_LED12.1 (VDD), R_LED13.1 (VDD), R_LED14.1 (VDD), R_LED15.1 (VDD), R_LED16.1 (VDD), R_LED17.1 (VDD), R_LED18.1 (VDD), R_LED19.1 (VDD), R_LED2.1 (VDD), R_LED20.1 (VDD), R_LED21.1 (VDD), R_LED22.1 (VDD), R_LED23.1 (VDD), R_LED24.1 (VDD), R_LED25.1 (VDD), R_LED26.1 (VDD), R_LED3.1 (VDD), R_LED4.1 (VDD), R_LED5.1 (VDD), R_LED6.1 (VDD), R_LED7.1 (VDD), R_LED8.1 (VDD), R_LED9.1 (VDD)
- net at L_D12.2 (A): now also L_SW12.2; no longer L_SW12.1
- net at L_D2.2 (A): now also L_SW2.2; no longer L_SW2.1
- net at L_D17.2 (A): now also L_SW17.2; no longer L_SW17.1
- net at L_D6.2 (A): now also L_SW6.2; no longer L_SW6.1
- net at L_D21.2 (A): now also L_SW21.2; no longer L_SW21.1
- net at L_D11.2 (A): now also L_SW11.2; no longer L_SW11.1
- net at L_D10.2 (A): now also L_SW10.2; no longer L_SW10.1
- net at L_D5.2 (A): now also L_SW5.2; no longer L_SW5.1
- net at L_D24.2 (A): now also L_SW24.2; no longer L_SW24.1
- net at L_D20.2 (A): now also L_SW20.2; no longer L_SW20.1
- net at L_D23.2 (A): now also L_SW23.2; no longer L_SW23.1
- net at L_D22.2 (A): now also L_SW22.2; no longer L_SW22.1
- net at L_D15.2 (A): now also L_SW15.2; no longer L_SW15.1
- net at L_D4.2 (A): now also L_SW4.2; no longer L_SW4.1
- net at L_D8.2 (A): now also L_SW8.2; no longer L_SW8.1
- net at L_D16.2 (A): now also L_SW16.2; no longer L_SW16.1
- net at L_LED1.2 (DOUT): now also L_LED2.4 (DIN)
- net at L_D26.2 (A): now also L_SW26.2; no longer L_SW26.1
- net at L_D13.2 (A): now also L_SW13.2; no longer L_SW13.1
- net at L_D14.2 (A): now also L_SW14.2; no longer L_SW14.1
- net at L_D19.2 (A): now also L_SW19.2; no longer L_SW19.1
- net at L_D18.2 (A): now also L_SW18.2; no longer L_SW18.1
- net at L_D1.2 (A): now also L_SW1.2; no longer L_SW1.1
- net at L_D25.2 (A): now also L_SW25.2; no longer L_SW25.1
- net at L_D7.2 (A): now also L_SW7.2; no longer L_SW7.1
- net at L_D9.2 (A): now also L_SW9.2; no longer L_SW9.1
- net at L_D3.2 (A): now also L_SW3.2; no longer L_SW3.1
- net at R_LED1.2 (DOUT): now also R_LED2.4 (DIN)
- new net: R_LED7.2 (DOUT), R_LED8.4 (DIN)
- new net: R_LED6.2 (DOUT), R_LED7.4 (DIN)
- new net: R_D22.2 (A), R_SW22.2
- new net: L_LED16.2 (DOUT), L_LED17.4 (DIN)
- new net: L_LED15.2 (DOUT), L_LED16.4 (DIN)
- new net: L_LED17.2 (DOUT), L_LED18.4 (DIN)
- new net: R_D7.2 (A), R_SW7.2
- new net: R_LED22.2 (DOUT), R_LED23.4 (DIN)
- new net: R_LED21.2 (DOUT), R_LED22.4 (DIN)
- new net: L_LED7.2 (DOUT), L_LED8.4 (DIN)
- new net: L_LED6.2 (DOUT), L_LED7.4 (DIN)
- new net: R_LED25.2 (DOUT), R_LED26.4 (DIN)
- new net: R_LED24.2 (DOUT), R_LED25.4 (DIN)
- new net: R_LED3.2 (DOUT), R_LED4.4 (DIN)
- new net: R_LED2.2 (DOUT), R_LED3.4 (DIN)
- new net: R_LED5.2 (DOUT), R_LED6.4 (DIN)
- new net: R_LED4.2 (DOUT), R_LED5.4 (DIN)
- new net: R_D9.2 (A), R_SW9.2
- new net: R_D15.2 (A), R_SW15.2
- new net: L_LED2.2 (DOUT), L_LED3.4 (DIN)
- new net: L_LED24.2 (DOUT), L_LED25.4 (DIN)
- new net: L_LED23.2 (DOUT), L_LED24.4 (DIN)
- new net: L_LED5.2 (DOUT), L_LED6.4 (DIN)
- new net: R_D20.2 (A), R_SW20.2
- new net: R_D11.2 (A), R_SW11.2
- new net: R_LED17.2 (DOUT), R_LED18.4 (DIN)
- new net: R_LED16.2 (DOUT), R_LED17.4 (DIN)
- new net: R_D21.2 (A), R_SW21.2
- new net: R_D26.2 (A), R_SW26.2
- new net: R_LED15.2 (DOUT), R_LED16.4 (DIN)
- new net: R_LED13.2 (DOUT), R_LED14.4 (DIN)
- new net: R_LED12.2 (DOUT), R_LED13.4 (DIN)
- new net: R_LED11.2 (DOUT), R_LED12.4 (DIN)
- new net: R_LED10.2 (DOUT), R_LED11.4 (DIN)
- new net: L_LED12.2 (DOUT), L_LED13.4 (DIN)
- new net: L_LED11.2 (DOUT), L_LED12.4 (DIN)
- new net: L_LED10.2 (DOUT), L_LED11.4 (DIN)
- new net: L_LED10.4 (DIN), L_LED9.2 (DOUT)
- new net: R_D2.2 (A), R_SW2.2
- new net: R_D5.2 (A), R_SW5.2
- new net: R_D18.2 (A), R_SW18.2
- new net: R_D3.2 (A), R_SW3.2
- new net: L_LED4.2 (DOUT), L_LED5.4 (DIN)
- new net: L_LED3.2 (DOUT), L_LED4.4 (DIN)
- new net: L_LED13.2 (DOUT), L_LED14.4 (DIN)
- new net: R_LED14.2 (DOUT), R_LED15.4 (DIN)
- new net: R_D17.2 (A), R_SW17.2
- new net: R_D6.2 (A), R_SW6.2
- new net: L_LED22.2 (DOUT), L_LED23.4 (DIN)
- new net: R_D10.2 (A), R_SW10.2
- new net: R_D13.2 (A), R_SW13.2
- new net: R_D4.2 (A), R_SW4.2
- new net: L_LED8.2 (DOUT), L_LED9.4 (DIN)
- new net: L_LED19.2 (DOUT), L_LED20.4 (DIN)
- new net: L_LED18.2 (DOUT), L_LED19.4 (DIN)
- new net: R_D24.2 (A), R_SW24.2
- new net: R_D16.2 (A), R_SW16.2
- new net: R_LED23.2 (DOUT), R_LED24.4 (DIN)
- new net: R_D19.2 (A), R_SW19.2
- new net: R_D1.2 (A), R_SW1.2
- new net: R_LED10.4 (DIN), R_LED9.2 (DOUT)
- new net: R_LED8.2 (DOUT), R_LED9.4 (DIN)
- new net: L_LED21.2 (DOUT), L_LED22.4 (DIN)
- new net: L_LED20.2 (DOUT), L_LED21.4 (DIN)
- new net: L_LED14.2 (DOUT), L_LED15.4 (DIN)
- new net: R_D12.2 (A), R_SW12.2
- new net: R_LED18.2 (DOUT), R_LED19.4 (DIN)
- new net: R_D23.2 (A), R_SW23.2
- new net: L_LED25.2 (DOUT), L_LED26.4 (DIN)
- new net: R_LED20.2 (DOUT), R_LED21.4 (DIN)
- new net: R_LED19.2 (DOUT), R_LED20.4 (DIN)
- new net: R_D25.2 (A), R_SW25.2
- new net: R_D8.2 (A), R_SW8.2
Other:
- moved on the sheet: BAT_EXT_L1, BAT_EXT_R1, BAT_L1, BAT_L2, BAT_R1, BAT_R2, C5, C6, C7, C8, H_L1, H_L2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

Commit message: - Routed most of diode-switch-caps tracks
Parts:
- renumbered L_D6 to L_D1, L_D18 to L_D13, L_D17 to L_D14, L_D16 to L_D15, L_D15 to L_D16, L_D14 to L_D17, L_D13 to L_D18, L_D5 to L_D2, L_D4 to L_D3, L_D3 to L_D4, L_D2 to L_D5, L_D1 to L_D6, L_SW6 to L_SW1, L_SW18 to L_SW13, L_SW17 to L_SW14, L_SW16 to L_SW15, L_SW15 to L_SW16, L_SW14 to L_SW17, L_SW13 to L_SW18, L_SW5 to L_SW2, L_SW4 to L_SW3, L_SW3 to L_SW4, L_SW2 to L_SW5, L_SW1 to L_SW6, R_D9 to R_D10, R_D8 to R_D11, R_D7 to R_D12, R_D26 to R_D19, R_D25 to R_D20, R_D24 to R_D21, R_D23 to R_D22, R_D22 to R_D23, R_D21 to R_D24, R_D20 to R_D25, R_D19 to R_D26, R_D12 to R_D7, R_D11 to R_D8, R_D10 to R_D9, R_SW9 to R_SW10, R_SW8 to R_SW11, R_SW7 to R_SW12, R_SW26 to R_SW19, R_SW25 to R_SW20, R_SW24 to R_SW21, R_SW23 to R_SW22, R_SW22 to R_SW23, R_SW21 to R_SW24, R_SW20 to R_SW25, R_SW19 to R_SW26, R_SW12 to R_SW7, R_SW11 to R_SW8, R_SW10 to R_SW9
Connections:
- net at R_D14.2 (A): now also R_SW14.2

Commit message: added more components and fix some in sch
Parts:
- added L_R1, L_R2, R_R1, R_R2: 10k, Resistor_SMD:R_0805_2012Metric, symbol Device:R
- added R_C5, R_C6: 10uf, Capacitor_SMD:C_0805_2012Metric, symbol Device:C_Small
- added R_J1, R_J2: Qwiic_RA, SparkFun-Connector:JST_SMD_1.0mm-4_RA, symbol SparkFun-Connector:Qwiic_Right_Angle
- renumbered C5 to R_C1, C6 to R_C2, C7 to R_C3, C8 to R_C4, TRRS_R1 to R_TRRS1, TRRS_R2 to R_TRRS2
Connections:
- net GND: now also R_C5.2, R_J1.1 (Pin_1), R_J2.1 (Pin_1)
- net GND2: now also R_C6.2
- net LED_OUT_R: no longer T-Display-S3_R1.3 (2)
- net R_SCL: now also R_J1.4 (Pin_4), R_J2.4 (Pin_4)
- net R_SDA: now also R_J1.3 (Pin_3), R_J2.3 (Pin_3)
- net at IO_R1.20 (~{RESET}): now also R_R2.2
- net at JP_R1.2 (B), R_TRRS1.1, R_TRRS2.1: now also R_J1.2 (Pin_2), R_J2.2 (Pin_2)
- net at IO_L1.20 (~{RESET}): now also L_R2.2
- net +3.3V_LEFT renamed +3.3V
- net +3.3V: now also L_R1.1, L_R2.1, R_C6.1
- net +3.3V_RIGHT renamed +3.3VA
- net +3.3VA: now also R_C5.1, R_R1.1, R_R2.1
- net +5V_LEFT renamed +5V
- net +5V_RIGHT renamed +5VA
- net IO_INT_L renamed L_IO_INT
- net L_IO_INT: now also L_R1.2
- net IO_INT_R renamed R_IO_INT
- net R_IO_INT: now also R_R1.2
- net VBAT_R renamed R_VBAT
- net VLED_R renamed R_VLED
- new net: R_J2.NC1 (NC), R_J2.NC2 (NC)
- new net: R_J1.NC1 (NC), R_J1.NC2 (NC)
- new net R_LED_OUT: T-Display-S3_R1.3 (2)
Other:
- moved on the sheet: IO_R1, JP_R1, R_C1, R_C2, R_C3, R_C4, R_TRRS1, R_TRRS2

Commit message: Right side almost done
Parts:
- removed R_J2: Qwiic_RA, SparkFun-Connector:JST_SMD_1.0mm-4_RA, symbol SparkFun-Connector:Qwiic_Right_Angle
- removed R_TRRS2, TRRS_L2: PRT-12639, Keebio:TRRS-PJ-320A, symbol TRRS:PRT-12639
- added L_J1: Qwiic_RA, SparkFun-Connector:JST_SMD_1.0mm-4_RA, symbol SparkFun-Connector:Qwiic_Right_Angle
- renumbered R_C6 to L_C5
Connections:
- net GND2: now also L_J1.1 (Pin_1)
- net L_SCL: now also L_J1.4 (Pin_4)
- net L_SDA: now also L_J1.3 (Pin_3)
- net at JP_L1.2 (B), TRRS_L1.1: now also L_J1.2 (Pin_2)
- new net: L_J1.NC1 (NC), L_J1.NC2 (NC)
Other:
- moved on the sheet: C1, C2, C3, C4

Commit message: -Almost done
Parts:
- R_TRRS1, TRRS_L1: footprint Keebio:TRRS-PJ-320A -> custom:TRRS-PJ-320A
Connections:
- net +3.3V: now also T-Display-S3_L1.1 (3v)
- net L_KEY_COL1: now also L_SW26.1; no longer L_SW25.1
- net L_KEY_COL2: now also L_SW25.1; no longer L_SW1.1, L_SW12.1, L_SW13.1, L_SW24.1
- net L_KEY_COL3: now also L_SW1.1, L_SW12.1, L_SW13.1, L_SW24.1; no longer L_SW11.1, L_SW14.1, L_SW2.1, L_SW23.1
- net L_KEY_COL4: now also L_SW11.1, L_SW14.1, L_SW2.1, L_SW23.1; no longer L_SW10.1, L_SW15.1, L_SW22.1, L_SW3.1
- net L_KEY_COL5: now also L_SW10.1, L_SW15.1, L_SW22.1, L_SW3.1; no longer L_SW16.1, L_SW21.1, L_SW4.1, L_SW9.1
- net L_KEY_COL6: now also L_SW16.1, L_SW21.1, L_SW4.1, L_SW9.1; no longer L_SW17.1, L_SW20.1, L_SW5.1, L_SW8.1
- net L_KEY_COL7: now also L_SW17.1, L_SW20.1, L_SW5.1, L_SW8.1; no longer L_SW18.1, L_SW19.1, L_SW6.1, L_SW7.1
- net L_KEY_COL8: now also L_SW18.1, L_SW19.1, L_SW6.1, L_SW7.1; no longer L_SW26.1
- no-connect marks 29 -> 28

Commit message: added outline and holes
Parts:
- renumbered BAT_L1 to L_BAT1, BAT_L2 to L_BAT2, BAT_EXT_L1 to L_BAT_EXT1, C1 to L_C1, C2 to L_C2, C3 to L_C3, C4 to L_C4, IO_L1 to L_IO1, IOExp_Pinout_L1 to L_IOExp_Pinout1, JP_L1 to L_JP1, JP_L2 to L_JP2, S3_Pinout_L1 to L_S3_Pinout1, SW_L1 to L_SWB1, T-Display-S3_L1 to L_T-Display-S3, BAT_R1 to R_BAT1, BAT_R2 to R_BAT2, BAT_EXT_R1 to R_BAT_EXT1, IO_R1 to R_IO1, IOExp_Pinout_R1 to R_IOExp_Pinout1, JP_R1 to R_JP1, JP_R2 to R_JP2, S3_Pinout_R1 to R_S3_Pinout1, SW_R1 to R_SWB1, T-Display-S3_R1 to R_T-Display-S3
Connections:
- net LED_OUT_R is gone; now on net R_LED_OUT: R_LED1.4 (DIN)
- net +3.3V renamed L_+3.3V
- net +3.3VA renamed R_+3.3V
- net +5V renamed L_+5V
- net +5VA renamed R_+5V
- net GND renamed R_GND
- net GND1 renamed R_GND1
- net GND2 renamed L_GND
- net GND3 renamed L_GND1
- net LED_OUT_L renamed L_LED_OUT
- net VBAT_L renamed L_VBAT
- net VLED_L renamed L_VLED

Commit message: holes located, kinda ready to send to production
Connections:
- net L_GND1 is gone; now on net L_GND: L_S3_Pinout1.10 (Pin_10), L_T-Display-S3.11 (GND)
- net R_GND1 is gone; now on net R_GND: R_S3_Pinout1.10 (Pin_10), R_T-Display-S3.11 (GND)
