File: split_keyboard.kicad_sch (KiCad schematic)
At the start: 204 parts

Commit message: Added all TPs
Parts:
- added L_BAT_EXT2, R_BAT_EXT2: Conn_01x02_Socket, Connector_PinHeader_2.54mm:PinHeader_1x02_P2.54mm_Vertical, symbol Connector:Conn_01x02_Socket
- added L_JP3, L_JP4, R_JP3, R_JP4: Measure, SparkFun-Jumper:Jumper_2_NC_Trace_NoSilk, symbol SparkFun-Jumper:Jumper_Measure
- added L_TP_GND1, L_TP_INT1, L_TP_LEDOUT1, L_TP_RST1, L_TP_VCC1, R_TP_GND1, R_TP_INT1, R_TP_LEDOUT1, R_TP_RST1, R_TP_VCC1: 1.25mm, SparkFun-Connector:TestPoint-1.25mm, symbol SparkFun-Connector:TestPoint_1.25mm
Connections:
- net L_GND: now also L_TP_GND1.1
- net L_IO_INT: now also L_TP_INT1.1
- net L_LED_OUT: now also L_TP_LEDOUT1.1
- net L_SCL: now also L_JP4.1 (A); no longer L_T-Display-S3.16 (44)
- net L_SDA: now also L_JP3.1 (A); no longer L_T-Display-S3.15 (43)
- net L_VBAT: now also L_BAT_EXT2.1 (Pin_1)
- net L_VLED: now also L_TP_VCC1.1
- net R_GND: now also R_TP_GND1.1
- net R_IO_INT: now also R_TP_INT1.1
- net R_LED_OUT: now also R_TP_LEDOUT1.1
- net R_SCL: now also R_JP4.1 (A); no longer R_T-Display-S3.16 (44)
- net R_SDA: now also R_JP3.1 (A); no longer R_T-Display-S3.15 (43)
- net R_VBAT: now also R_BAT_EXT2.1 (Pin_1)
- net R_VLED: now also R_TP_VCC1.1
- net at R_BAT1.2 (Pin_2), R_BAT2.2 (Pin_2), R_BAT_EXT1.2 (Pin_2): now also R_BAT_EXT2.2 (Pin_2)
- net at L_IO1.20 (~{RESET}), L_R2.2: now also L_TP_RST1.1
- net at R_IO1.20 (~{RESET}), R_R2.2: now also R_TP_RST1.1
- net at L_BAT1.2 (Pin_2), L_BAT2.2 (Pin_2), L_BAT_EXT1.2 (Pin_2): now also L_BAT_EXT2.2 (Pin_2)
- new net: L_JP4.2 (B), L_T-Display-S3.16 (44)
- new net: R_JP4.2 (B), R_T-Display-S3.16 (44)
- new net: R_JP3.2 (B), R_T-Display-S3.15 (43)
- new net: L_JP3.2 (B), L_T-Display-S3.15 (43)
Other:
- moved on the sheet: L_BAT1, L_BAT2, L_R1, L_R2, L_SWB1, L_T-Display-S3, R_C5, R_T-Display-S3

Commit message: Finished board with plates done.
Parts:
- added H_L6, H_R6: MountingHole, MountingHole:MountingHole_2.5mm_Pad_TopBottom, symbol Mechanical:MountingHole
Changed lines of the file:
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@@
+	)
+	(symbol
+		(lib_id "Mechanical:MountingHole")
+		(at 629.92 274.32 0)
+		(unit 1)
+		(exclude_from_sim no)
+		(in_bom yes)
+		(on_board yes)
+		(dnp no)
+		(fields_autoplaced yes)
+		(property "Reference" "H_R6"
+			(at 632.46 273.0499 0)
+			(effects
+				(font
+					(size 1.27 1.27)
+				)
+				(justify left)
+			)
+		)
+		(property "Value" "MountingHole"
+			(at 632.46 275.5899 0)
+			(effects
+				(font
+					(size 1.27 1.27)
+				)
+				(justify left)
+			)
+		)
+		(property "Footprint" "MountingHole:MountingHole_2.5mm_Pad_TopBottom"
+			(at 629.92 274.32 0)
+			(effects
+				(font
+					(size 1.27 1.27)
+				)
+				(hide yes)
+			)
+		)
+		(property "Datasheet" "~"
+			(at 629.92 274.32 0)
+			(effects
+				(font
+					(size 1.27 1.27)
+				)
+				(hide yes)
+			)
+		)
+		(property "Description" ""
+			(at 629.92 274.32 0)
+			(effects
+				(font
+					(size 1.27 1.27)
+				)
+				(hide yes)
+			)
+		)
+		(instances
+			(project "split_keyboard"
+				(path "/48c5ed27-feda-4a94-9dac-8f2f8efef842"
+					(reference "H_R6")
+					(unit 1)
+				)
+			)
+		)
 	)
 	(symbol
@@
 					(unit 1)
 				)
+			)
+		)
+	)
+	(symbol
+		(lib_id "Mechanical:MountingHole")
+		(at 185.42 266.7 0)
+		(unit 1)
+		(exclude_from_sim no)
+		(in_bom yes)
+		(on_board yes)
+		(dnp no)
+		(fields_autoplaced yes)
+		(property "Reference" "H_L6"
+			(at 187.96 265.4299 0)
+			(effects
+				(font
+					(size 1.27 1.27)
+				)
+				(justify left)
+			)
+		)
+		(property "Value" "MountingHole"
+			(at 187.96 267.9699 0)
+			(effects
+				(font
+					(size 1.27 1.27)
+				)
+				(justify left)
+			)
+		)
+		(property "Footprint" "MountingHole:MountingHole_2.5mm_Pad_TopBottom"
+			(at 185.42 266.7 0)
+			(effects
+				(font
+					(size 1.27 1.27)
+				)
+				(hide yes)
+			)
+		)
+		(property "Datasheet" "~"
+			(at 185.42 266.7 0)
+			(effects
+				(font
+					(size 1.27 1.27)
+				)
+				(hide yes)
+			)
+		)
+		(property "Description" ""
+			(at 185.42 266.7 0)
+			(effects
+				(font
+					(size 1.27 1.27)
+				)
+				(hide yes)
+			)
+		)
+		(instances
+			(project "split_keyboard"
+				(path "/48c5ed27-feda-4a94-9dac-8f2f8efef842"
+					(reference "H_L6")
+					(unit 1)
+				)
